File: st32.brd (EAGLE design)
At the start: 160 x 100 mm, 30 parts, among them Q1 26MHz, U1 STM32F407IGT6

Commit message: power
Parts:
- added C25: 100µ, resistor:E2,5-6
- added C26: 1000µ, resistor:E5-13
- added C27, C28, C29: 100nF, resistor:C1206
- added CN1: (no value), adafruit:USB-MINIB
- added L2: 220µ, resistor:TJ3-U1
- added Q3, Q6: MOSFET-PGDS_TO220V, adafruit:TO220V
- added Q4, Q5, Q7, Q8: (no value), semicon-smd-ipc:SOT23
- added R2, R4: 10k, resistor:M1206
- added R3, R5: 47k, resistor:M1206
- added U$2: RPI-ZERO, RPI-Zero:RASPBERRYPI_BASTELSTUBE_V13_RASPI_BOARD_B+_FULL
- added U3: TSR_1-2433, 1_Robo-Lib:TSR-1
- moved D1 202.5 mm to (139.7, 15.2)
- moved R1 192.3 mm to (134.6, 8.89)
- moved C23 184.1 mm to (134.6, 3.81)
- moved U1 39.5 mm to (114.3, 30.5), turned to 180 degrees
Connections:
- net VBAT renamed V_BAT
- removed net GND: C1.2, C10.2, C11.2, C12.2, C13.2, C14.2, C15.2, C16.2, C17.2, C18.2, C19.2, C2.2, C20.2, C21.2, C22.2, C23.2, C24.2, C3.2, C4.2, C5.2, C6.2, C7.2, C8.2, C9.2, TS1.3, TS1.4, U$1.9, U1.102, U1.113, U1.126, U1.135, U1.14, U1.148, U1.158, U1.22, U1.37, U1.48, U1.61, U1.71, U1.90
- new net +14V: Q6.2, Q8.2
- new net +5V: CN1.VBUS, Q3.2, Q5.2
- new net D+: CN1.D+, U1.123
- new net D-: CN1.D-, U1.122
- new net GND2: C25.-, C26.-, C27.2, C28.2, C29.1, CN1.GND, R2.1, R3.1, R4.1, R5.1, U3.2
- new net GND_PWR: C1.2, C10.2, C11.2, C12.2, C13.2, C14.2, C15.2, C16.2, C17.2, C18.2, C19.2, C2.2, C20.2, C21.2, C22.2, C23.2, C24.2, C3.2, C4.2, C5.2, C6.2, C7.2, C8.2, C9.2, TS1.3, TS1.4, U$1.9, U$2.14, U$2.20, U$2.25, U$2.30, U$2.34, U$2.39, U$2.6, U$2.9, U1.102, U1.113, U1.126, U1.135, U1.14, U1.148, U1.158, U1.22, U1.37, U1.48, U1.61, U1.71, U1.90
- new net N$18: Q4.1, Q5.1, Q5.3, R2.2
- new net N$19: Q3.1, Q4.3, R3.2
- new net N$21: Q7.1, Q8.1, Q8.3, R4.2
- new net N$22: Q6.1, Q7.3, R5.2
- new net N$37: C29.2, L2.2, U3.3
- new net V_SUPPLY: C25.+, C28.1, Q3.3, Q4.2, Q6.3, Q7.2, U3.1
- net +3V3: now also C26.+, C27.1, L2.1, U$2.1, U$2.17

Commit message: Brushlesstreiber 1. Ansatz(brauchen wir das?;)
Parts:
- added C30: 100mF, resistor:C0603
- added C31, C33, C35: 220nF, resistor:C0805
- added C32, C34, C36: 100nF, resistor:C0805
- added D2, D3, D4: BAS21, diode:SOT23
- added R10, R11, R12, R13, R14, R6, R7, R8, R9: 47R, resistor:M0805
- added U$3, U$4, U$5, U$6, U$7, U$8: IRLR7843, eigenes:D-PACK
- added U2, U4, U5: IR2104STRPBF, ir2104:SOIC127P600X175-8N
- added X1: (no value), con-weidmueller-sl35:90-3
Connections:
- new net GND3: C32.2, C34.2, C36.2, U$4.2, U$6.2, U$8.2, U2.4, U4.4, U5.4
- new net IN_A: R8.2, U2.2
- new net IN_B: R14.2, U5.2
- new net IN_C: R11.2, U4.2
- new net N$2: R6.2, U$3.1
- new net N$20: C31.1, D2.3, U2.8
- new net N$23: R7.1, U2.5
- new net N$24: R6.1, U2.7
- new net N$25: R7.2, U$4.1
- new net N$26: C33.1, D3.3, U4.8
- new net N$27: R10.1, U4.5
- new net N$28: R9.1, U4.7
- new net N$29: R10.2, U$6.1
- new net N$30: R9.2, U$5.1
- new net N$31: C35.1, D4.3, U5.8
- new net N$32: R13.1, U5.5
- new net N$33: R12.1, U5.7
- new net N$34: R13.2, U$8.1
- new net N$35: R12.2, U$7.1
- new net PHASE_A: C31.2, U$3.2, U$4.3, U2.6, X1.1
- new net PHASE_B: C35.2, U$7.2, U$8.3, U5.6, X1.2
- new net PHASE_C: C33.2, U$5.2, U$6.3, U4.6, X1.3
- new net PWM_A: R8.1
- new net PWM_B: R14.1
- new net PWM_C: R11.1
- new net SD_A: U2.3
- new net SD_B: U5.3
- new net SD_C: U4.3
- net +14V: now also C32.1, C34.1, C36.1, D2.1, D3.1, D4.1, U$3.3, U$5.3, U$7.3, U2.1, U4.1, U5.1
- net +5V: now also C30.1
- net GND2: now also C30.2
