File: st32.sch (EAGLE design)
At the start: 30 parts, among them Q1 26MHz, U1 STM32F407IGT6

Commit message: power
Parts:
- added C25: 100µ, resistor:CPOL-EUE2.5-6
- added C26: 1000µ, resistor:CPOL-EUE5-13
- added C27, C28, C29: 100nF, resistor:C-EUC1206
- added CN1: (no value), adafruit:USBMINIB
- added L2: 220µ, resistor:L-EUTJ3-U1
- added Q3, Q6: MOSFET-PGDS_TO220V, adafruit:MOSFET-PGDS_TO220V
- added Q4, Q5, Q7, Q8: (no value), semicon-smd-ipc:PNP-TRANSISTOR_SOT23
- added R2, R4: 10k, resistor:R-EU_M1206
- added R3, R5: 47k, resistor:R-EU_M1206
- added U$2: RPI-ZERO, RPI-Zero:RPI-ZERO
- added U3: TSR_1-2433, 1_Robo-Lib:TSR_1-2433
Connections:
- net VBAT renamed V_BAT
- removed net GND: C1.2, C10.2, C11.2, C12.2, C13.2, C14.2, C15.2, C16.2, C17.2, C18.2, C19.2, C2.2, C20.2, C21.2, C22.2, C23.2, C24.2, C3.2, C4.2, C5.2, C6.2, C7.2, C8.2, C9.2, TS1.S, U$1.GND, U1A.BYPASS_REG, U1A.VSS, U1A.VSSA, U1A.VSS_2, U1A.VSS_3, U1A.VSS_4, U1B.VSS, U1B.VSS_2, U1B.VSS_3, U1B.VSS_4, U1B.VSS_5, U1B.VSS_6, U1B.VSS_7
- new net +14V: Q6.D, Q8.E
- new net +5V: CN1.VBUS, Q3.D, Q5.E
- new net D+: CN1.D+, U1B.PA12
- new net D-: CN1.D-, U1B.PA11
- new net GND2: C25.-, C26.-, C27.2, C28.2, C29.1, CN1.GND, R2.1, R3.1, R4.1, R5.1, U3.GND
- new net GND_PWR: C1.2, C10.2, C11.2, C12.2, C13.2, C14.2, C15.2, C16.2, C17.2, C18.2, C19.2, C2.2, C20.2, C21.2, C22.2, C23.2, C24.2, C3.2, C4.2, C5.2, C6.2, C7.2, C8.2, C9.2, TS1.S, U$1.GND, U$2.GND@1, U$2.GND@2, U$2.GND@3, U$2.GND@4, U$2.GND@5, U$2.GND@6, U$2.GND@7, U$2.GND@8, U1A.BYPASS_REG, U1A.VSS, U1A.VSSA, U1A.VSS_2, U1A.VSS_3, U1A.VSS_4, U1B.VSS, U1B.VSS_2, U1B.VSS_3, U1B.VSS_4, U1B.VSS_5, U1B.VSS_6, U1B.VSS_7
- new net N$18: Q4.B, Q5.B, Q5.C, R2.2
- new net N$19: Q3.G, Q4.C, R3.2
- new net N$21: Q7.B, Q8.B, Q8.C, R4.2
- new net N$22: Q6.G, Q7.C, R5.2
- new net N$37: C29.2, L2.2, U3.VO
- new net V_SUPPLY: C25.+, C28.1, Q3.S, Q4.E, Q6.S, Q7.E, U3.VI
- net +3V3: now also C26.+, C27.1, L2.1, U$2.3V3@1, U$2.3V3@2
Other:
- note added: "TRACO"
- note added: "USB"

Commit message: Brushlesstreiber 1. Ansatz(brauchen wir das?;)
Parts:
- added C30: 100mF, resistor:C-EUC0603
- added C31, C33, C35: 220nF, resistor:C-EUC0805
- added C32, C34, C36: 100nF, resistor:C-EUC0805
- added D2, D3, D4: BAS21, diode:ZENER-DIODESOT23
- added R10, R11, R12, R13, R14, R6, R7, R8, R9: 47R, resistor:R-EU_M0805
- added U$3, U$4, U$5, U$6, U$7, U$8: IRLR7843, eigenes:IRLR7843
- added U2, U4, U5: IR2104STRPBF, ir2104:IR2104STRPBF
- added X1: (no value), con-weidmueller-sl35:90-3
Connections:
- new net GND3: C32.2, C34.2, C36.2, U$4.S, U$6.S, U$8.S, U2.COM, U4.COM, U5.COM
- new net IN_A: R8.2, U2.IN
- new net IN_B: R14.2, U5.IN
- new net IN_C: R11.2, U4.IN
- new net N$2: R6.2, U$3.G
- new net N$20: C31.1, D2.C, U2.VB
- new net N$23: R7.1, U2.LO
- new net N$24: R6.1, U2.HO
- new net N$25: R7.2, U$4.G
- new net N$26: C33.1, D3.C, U4.VB
- new net N$27: R10.1, U4.LO
- new net N$28: R9.1, U4.HO
- new net N$29: R10.2, U$6.G
- new net N$30: R9.2, U$5.G
- new net N$31: C35.1, D4.C, U5.VB
- new net N$32: R13.1, U5.LO
- new net N$33: R12.1, U5.HO
- new net N$34: R13.2, U$8.G
- new net N$35: R12.2, U$7.G
- new net PHASE_A: C31.2, U$3.S, U$4.D, U2.VS, X1.1
- new net PHASE_B: C35.2, U$7.S, U$8.D, U5.VS, X1.2
- new net PHASE_C: C33.2, U$5.S, U$6.D, U4.VS, X1.3
- new net PWM_A: R8.1
- new net PWM_B: R14.1
- new net PWM_C: R11.1
- new net SD_A: U2.~SD
- new net SD_B: U5.~SD
- new net SD_C: U4.~SD
- net +14V: now also C32.1, C34.1, C36.1, D2.A, D3.A, D4.A, U$3.D, U$5.D, U$7.D, U2.VCC, U4.VCC, U5.VCC
- net +5V: now also C30.1
- net GND2: now also C30.2
Other:
- note added: "Brushlesstreiber No.1"
- note added: "ESP-8266"
- note added: "Pasberry-PI ZERO"
- note added: "RESET-STM32"
- note added: "STM32"
- note added: "VBAT"
